File: gateway/knuth-gateway/knuth-gateway.kicad_pcb (KiCad board)
At the start: 2 copper layers, 12 parts, among them U1 FONA808, U2 Q_RHS, U3 CUI_5V_SWITCHING, U4 tpl5110, U5 adasolarlipo, U7 powerboost_500

Commit message: update
Parts:
- added J1: Conn_01x16_Female, Connector_PinSocket_2.54mm:PinSocket_1x16_P2.54mm_Vertical, F.Cu at (214.6, 106.7)
- added Q1: Q_NPN_EBC, Package_TO_SOT_THT:TO-92, F.Cu at (231.1, 86.4)
- added Q2: Q_NPN_BCE, Package_TO_SOT_THT:TO-220-3_Vertical, F.Cu at (238.8, 100.3)
- moved R2 23.4 mm to (240.0, 76.2)
- moved R_Delay1 15.9 mm to (243.8, 99.1), turned to 90 degrees
- moved R3 15.3 mm to (241.3, 87.6), turned to 0 degrees
- moved U5 12.0 mm to (246.4, 78.7), turned to 180 degrees
- moved U4 8.98 mm to (254.0, 88.9)
- moved J_DC_6V_IN1 7.73 mm to (254.0, 71.1)
- moved J_DC_6.5V+_IN1 7.73 mm to (254.0, 77.5)
- moved R1 5.24 mm to (232.4, 94.0)
- moved U2 3.81 mm to (219.7, 106.7)
Routing:
- net Net-(J1-Pad13): track 0.00 -> 129.2 mm
- net Net-(J1-Pad1): track 0.00 -> 127.0 mm, vias 0 -> 2
- net GND: track 0.00 -> 116.4 mm, vias 0 -> 8
- net Net-(J1-Pad11): track 0.00 -> 59.0 mm
- net Net-(Q2-Pad2): track 0.00 -> 48.7 mm, vias 0 -> 2
- net Net-(J1-Pad12): track 0.00 -> 47.5 mm
- net Net-(J_DC_6.5V+_IN1-Pad1): track 0.00 -> 41.7 mm, vias 0 -> 2
- net +BATT: track 0.00 -> 41.3 mm, vias 0 -> 2
- net Net-(J_DC_6V_IN1-Pad1): track 0.00 -> 16.1 mm
- net Net-(Q1-Pad2): track 0.00 -> 12.0 mm
- net Net-(J1-Pad3): track 0.00 -> 11.4 mm, vias 0 -> 2
- net Net-(Q2-Pad1): track 0.00 -> 11.2 mm
- net Net-(R_Delay1-Pad2): track 0.00 -> 10.5 mm
- net Net-(R2-Pad1): track 0.00 -> 9.47 mm
- net Net-(J1-Pad9): track 0.00 -> 5.08 mm
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Other:
- board outline added: 66.7 x 61.6 mm
- net class Default: via_dia 0.8 -> 1.778; via_drill 0.4 -> 0.889
- rule via_min_drill: 0.3 -> 0.508
- board text added: "Knuth Ranch: Cellular Adapter"
- board text added: "pvos.org/knuth"

Commit message: update
Parts:
- Q2: value Q_NPN_BCE -> Q_PNP_BCE; footprint Package_TO_SOT_THT:TO-220-3_Vertical -> TO_SOT_Packages_THT:TO-220-3_Vertical
- moved R_Delay1 9.65 mm to (248.8, 90.8), turned to 0 degrees
- moved Q2 8.93 mm to (236.6, 91.7), turned to 270 degrees
- moved Q1 5.39 mm to (235.2, 82.8), turned to 270 degrees
- moved R3 1.41 mm to (240.0, 87.1)
- moved R1 1.24 mm to (231.6, 93.0)
Connections:
- Q1 pad 1: Net-(Q1-Pad1) -> GND
- Q1 pad 3: GND -> Net-(Q1-Pad3)
- R1 pad 2: Net-(Q1-Pad1) -> Net-(Q1-Pad3)
- U1 pad 1: Net-(U1-Pad1) -> (no net)
- U1 pad 10: Net-(U1-Pad10) -> (no net)
- U1 pad 11: Net-(U1-Pad11) -> (no net)
- U1 pad 12: Net-(U1-Pad12) -> (no net)
- U1 pad 13: Net-(U1-Pad13) -> (no net)
- U1 pad 14: Net-(U1-Pad14) -> (no net)
- U1 pad 15: Net-(U1-Pad15) -> (no net)
- U1 pad 16: Net-(U1-Pad16) -> (no net)
- U1 pad 5: Net-(U1-Pad5) -> (no net)
- U1 pad 8: Net-(U1-Pad8) -> (no net)
- U7 pad 1: Net-(U7-Pad1) -> (no net)
- U7 pad 4: Net-(U7-Pad4) -> (no net)
- U7 pad 5: Net-(U7-Pad5) -> (no net)
- U7 pad 6: Net-(U7-Pad6) -> (no net)
- U7 pad 7: Net-(U7-Pad7) -> (no net)
Routing:
- net Net-(R3-Pad2): track 0.00 -> 23.5 mm
- net Net-(J1-Pad3): track 11.4 -> 30.9 mm, vias 2 -> 0
- net Net-(Q2-Pad2): track 48.7 -> 59.8 mm, vias 2 -> 0
- net Net-(Q1-Pad2): track 12.0 -> 5.17 mm
- net Net-(Q2-Pad1): track 11.2 -> 5.54 mm
- net Net-(R_Delay1-Pad2): track 10.5 -> 5.45 mm
- net Net-(Q1-Pad3): track 0.00 -> 4.71 mm
- net GND: track 116.4 -> 120.4 mm
- net Net-(Q1-Pad1): track 3.07 -> 0.00 mm
- net Net-(J1-Pad13): track 129.2 -> 132.0 mm
- net Net-(J1-Pad1): track 127.0 -> 129.5 mm
- net Net-(J1-Pad11): track 59.0 -> 56.7 mm, vias 0 -> 2
- net +BATT: track 41.3 -> 43.5 mm
- net Net-(J1-Pad12): track 47.5 -> 47.0 mm, vias 0 -> 2
