File: gateway/knuth-gateway/knuth-gateway.sch (KiCad schematic (older format))
At the start: 15 parts, among them Q1 Q_NPN_EBC, Q2 Q_NPN_BCE

Commit message: update
Parts:
- removed U?: adasolarlipo, symbol knuth:adasolarlipo
- added J?: Conn_01x16_Female, symbol Connector:Conn_01x16_Female
- J_DC_6.5V+_IN1: renamed from J_DC_6.5V+_IN; footprint (none) -> Connector_PinSocket_2.54mm:PinSocket_1x02_P2.54mm_Vertical
- J_DC_6V_IN1: renamed from J_DC_6V_IN; footprint (none) -> Connector_PinSocket_2.54mm:PinSocket_1x02_P2.54mm_Vertical
- R1: footprint (none) -> Resistor_THT:R_Axial_DIN0204_L3.6mm_D1.6mm_P5.08mm_Horizontal
- R2, R3: renamed from R?; footprint (none) -> Resistor_THT:R_Axial_DIN0204_L3.6mm_D1.6mm_P5.08mm_Horizontal
- R_Delay1: renamed from R_Delay; footprint (none) -> Connector_PinSocket_2.54mm:PinSocket_1x02_P2.54mm_Vertical
- U1, U2: renamed from U?; footprint (none) -> Connector_PinSocket_2.54mm:PinSocket_1x16_P2.54mm_Vertical
- U3: renamed from U?; footprint (none) -> Connector_PinSocket_2.54mm:PinSocket_1x03_P2.54mm_Vertical
- U4: renamed from U?; footprint (none) -> Connector_PinSocket_2.54mm:PinSocket_1x05_P2.54mm_Vertical
- U5: renamed from U?; footprint (none) -> Connector_PinSocket_2.54mm:PinSocket_1x04_P2.54mm_Vertical
- U7: renamed from U?; footprint (none) -> Connector_PinSocket_2.54mm:PinSocket_1x08_P2.54mm_Vertical
Connections:
- net GND: now also J?.7 (Pin_7)
- net at U1.4 (Vio), U2.3 (3v3): now also J?.3 (Pin_3)
- net at U1.6 (RX), U2.12 (21): now also J?.12 (Pin_12)
- net at U1.7 (TX), U2.11 (19): now also J?.11 (Pin_11)
- net at U2.13 (22), U4.5 (Done): now also J?.13 (Pin_13)
- net at U2.1 (VIN), U7.8 (5V): now also J?.1 (Pin_1)
- net at U2.10 (18): now also J?.10 (Pin_10)
- net at U2.14 (23): now also J?.14 (Pin_14)
- net at U2.15 (35): now also J?.15 (Pin_15)
- net at U2.16 (RST): now also J?.16 (Pin_16)
- net at U2.2 (5V): now also J?.2 (Pin_2)
- net at U2.4 (2): now also J?.4 (Pin_4)
- net at U2.5 (12): now also J?.5 (Pin_5)
- net at U2.6 (14): now also J?.6 (Pin_6)
- net at U2.8 (0): now also J?.8 (Pin_8)
- net at U2.9 (5): now also J?.9 (Pin_9)
Changed lines of the file:
@@
 F 0 "R1" H 5370 4046 50  0000 L CNN
 F 1 "R" H 5370 3955 50  0000 L CNN
-F 2 "" V 5230 4000 50  0001 C CNN
+F 2 "Resistor_THT:R_Axial_DIN0204_L3.6mm_D1.6mm_P5.08mm_Horizontal" V 5230 4000 50  0001 C CNN
 F 3 "~" H 5300 4000 50  0001 C CNN
 	1    5300 4000
@@
 $EndComp
 $Comp
-L knuth:FONA808 U?
+L knuth:FONA808 U1
 U 1 1 5D195B61
 P 1750 2600
-F 0 "U?" H 1706 3065 50  0000 C CNN
+F 0 "U1" H 1706 3065 50  0000 C CNN
 F 1 "FONA808" H 1706 2974 50  0000 C CNN
-F 2 "" H 1750 2600 50  0001 C CNN
+F 2 "Connector_PinSocket_2.54mm:PinSocket_1x16_P2.54mm_Vertical" H 1750 2600 50  0001 C CNN
 F 3 "" H 1750 2600 50  0001 C CNN
 	1    1750 2600
@@
 $EndComp
 $Comp
-L knuth:tpl5110 U?
+L knuth:tpl5110 U4
 U 1 1 5D196517
 P 3200 2500
-F 0 "U?" H 2956 2865 50  0000 C CNN
+F 0 "U4" H 2956 2865 50  0000 C CNN
 F 1 "tpl5110" H 2956 2774 50  0000 C CNN
-F 2 "" H 3200 2500 50  0001 C CNN
+F 2 "Connector_PinSocket_2.54mm:PinSocket_1x05_P2.54mm_Vertical" H 3200 2500 50  0001 C CNN
 F 3 "" H 3200 2500 50  0001 C CNN
 	1    3200 2500
@@
 $EndComp
 $Comp
-L power:+BATT #PWR?
+L power:+BATT #PWR0101
 U 1 1 5D19682C
 P 3450 2200
-F 0 "#PWR?" H 3450 2050 50  0001 C CNN
+F 0 "#PWR0101" H 3450 2050 50  0001 C CNN
 F 1 "+BATT" H 3465 2373 50  0000 C CNN
 F 2 "" H 3450 2200 50  0001 C CNN
@@
 	3200 2500 3500 2500
 $Comp
-L power:GND #PWR?
+L power:GND #PWR0102
 U 1 1 5D196982
 P 3750 2500
-F 0 "#PWR?" H 3750 2250 50  0001 C CNN
+F 0 "#PWR0102" H 3750 2250 50  0001 C CNN
 F 1 "GND" H 3755 2327 50  0000 C CNN
 F 2 "" H 3750 2500 50  0001 C CNN
@@
 	3300 2400 3450 2400
 $Comp
-L knuth:adasolarlipo U?
+L knuth:adasolarlipo U5
 U 1 1 5D196E31
 P 4100 1950
-F 0 "U?" H 3823 2046 50  0000 R CNN
+F 0 "U5" H 3823 2046 50  0000 R CNN
 F 1 "adasolarlipo" H 3823 1955 50  0000 R CNN
-F 2 "" H 4100 1950 50  0001 C CNN
+F 2 "Connector_PinSocket_2.54mm:PinSocket_1x04_P2.54mm_Vertical" H 4100 1950 50  0001 C CNN
 F 3 "" H 4100 1950 50  0001 C CNN
 	1    4100 1950
@@
 	1950 2600 2500 2600
 $Comp
-L Connector:Conn_01x02_Female R_Delay
+L Connector:Conn_01x02_Female R_Delay1
 U 1 1 5D197A39
 P 4800 2600
-F 0 "R_Delay" H 4827 2576 50  0000 L CNN
+F 0 "R_Delay1" H 4827 2576 50  0000 L CNN
 F 1 "Conn_01x02_Female" H 4827 2485 50  0000 L CNN
-F 2 "" H 4800 2600 50  0001 C CNN
+F 2 "Connector_PinSocket_2.54mm:PinSocket_1x02_P2.54mm_Vertical" H 4800 2600 50  0001 C CNN
 F 3 "~" H 4800 2600 50  0001 C CNN
 	1    4800 2600
@@
 	3400 2800 4600 2800
 $Comp
-L Device:R R?
+L Device:R R3
 U 1 1 5D198BCF
 P 4050 3300
-F 0 "R?" V 3843 3300 50  0000 C CNN
+F 0 "R3" V 3843 3300 50  0000 C CNN
 F 1 "R" V 3934 3300 50  0000 C CNN
-F 2 "" V 3980 3300 50  0001 C CNN
+F 2 "Resistor_THT:R_Axial_DIN0204_L3.6mm_D1.6mm_P5.08mm_Horizontal" V 3980 3300 50  0001 C CNN
 F 3 "~" H 4050 3300 50  0001 C CNN
 	1    4050 3300
@@
 	4700 3550 4700 3350
 $Comp
-L power:+BATT #PWR?
+L power:+BATT #PWR0103
 U 1 1 5D199524
 P 4700 3350
-F 0 "#PWR?" H 4700 3200 50  0001 C CNN
+F 0 "#PWR0103" H 4700 3200 50  0001 C CNN
 F 1 "+BATT" H 4715 3523 50  0000 C CNN
 F 2 "" H 4700 3350 50  0001 C CNN
@@
 	4200 4350 5000 4350
 $Comp
-L knuth:powerboost_500 U?
+L knuth:powerboost_500 U7
 U 1 1 5D19A756
 P 6900 3700
-F 0 "U?" H 6423 3604 50  0000 R CNN
+F 0 "U7" H 6423 3604 50  0000 R CNN
 F 1 "powerboost_500" H 6423 3695 50  0000 R CNN
-F 2 "" H 6900 3700 50  0001 C CNN
+F 2 "Connector_PinSocket_2.54mm:PinSocket_1x08_P2.54mm_Vertical" H 6900 3700 50  0001 C CNN
 F 3 "" H 6900 3700 50  0001 C CNN
 	1    6900 3700
@@
 	5500 3550 6100 3550
 $Comp
-L power:GND #PWR?
+L power:GND #PWR0104
 U 1 1 5D19AE89
 P 6550 4000
-F 0 "#PWR?" H 6550 3750 50  0001 C CNN
+F 0 "#PWR0104" H 6550 3750 50  0001 C CNN
 F 1 "GND" H 6555 3827 50  0000 C CNN
 F 2 "" H 6550 4000 50  0001 C CNN
@@
 	6550 3900 6550 4000
 $Comp
-L knuth:Q_RHS U?
+L knuth:Q_RHS U2
 U 1 1 5D19C257
 P 1750 5600
-F 0 "U?" H 1681 6865 50  0000 C CNN
+F 0 "U2" H 1681 6865 50  0000 C CNN
 F 1 "Q_RHS" H 1681 6774 50  0000 C CNN
-F 2 "" H 1750 5600 50  0001 C CNN
+F 2 "Connector_PinSocket_2.54mm:PinSocket_1x16_P2.54mm_Vertical" H 1750 5600 50  0001 C CNN
 F 3 "" H 1750 5600 50  0001 C CNN
 	1    1750 5600
@@
 	2100 3200 2100 3350
 $Comp
-L power:GND #PWR?
+L power:GND #PWR0105
 U 1 1 5D19CDAE
 P 2100 3350
-F 0 "#PWR?" H 2100 3100 50  0001 C CNN
+F 0 "#PWR0105" H 2100 3100 50  0001 C CNN
 F 1 "GND" H 2105 3177 50  0000 C CNN
 F 2 "" H 2100 3350 50  0001 C CNN
@@
 	1850 5500 2400 5500
 $Comp
-L power:GND #PWR?
+L power:GND #PWR0106
 U 1 1 5D1A1ECD
 P 2400 5500
-F 0 "#PWR?" H 2400 5250 50  0001 C CNN
+F 0 "#PWR0106" H 2400 5250 50  0001 C CNN
 F 1 "GND" H 2405 5327 50  0000 C CNN
 F 2 "" H 2400 5500 50  0001 C CNN
@@
 Wire Wire Line
 	6400 3050 6400 6100
-$Comp
-L knuth:adasolarlipo U?
-U 1 1 5D1A87A3
-P 6300 2300
-F 0 "U?" H 6023 2304 50  0000 R CNN
-F 1 "adasolarlipo" H 6023 2395 50  0000 R CNN
-F 2 "" H 6300 2300 50  0001 C CNN
-F 3 "" H 6300 2300 50  0001 C CNN
-	1    6300 2300
-	-1   0    0    1
-$EndComp
-$Comp
-L power:GND #PWR?
-U 1 1 5D1A8823
-P 5850 2300
-F 0 "#PWR?" H 5850 2050 50  0001 C CNN
-F 1 "GND" H 5855 2127 50  0000 C CNN
-F 2 "" H 5850 2300 50  0001 C CNN
-F 3 "" H 5850 2300 50  0001 C CNN
-	1    5850 2300
-	1    0    0    -1
-$EndComp
-Wire Wire Line
-	6200 2300 5850 2300
 Wire Wire Line
 	4900 3550 4900 2950
-Wire Wire Line
-	4900 2950 6200 2950
-Wire Wire Line
-	6200 2950 6200 2400
 Connection ~ 4900 3550
 Wire Wire Line
 	4900 3550 4700 3550
 $Comp
-L power:GND #PWR?
+L power:GND #PWR0108
 U 1 1 5D1AA2EF
 P 5300 4550
-F 0 "#PWR?" H 5300 4300 50  0001 C CNN
+F 0 "#PWR0108" H 5300 4300 50  0001 C CNN
 F 1 "GND" H 5305 4377 50  0000 C CNN
 F 2 "" H 5300 4550 50  0001 C CNN
@@
 	4000 2150 3750 2150
 $Comp
-L Connector:Conn_01x02_Female J_DC_6V_IN
+L Connector:Conn_01x02_Female J_DC_6V_IN1
 U 1 1 5D1B33C1
 P 4400 1350
-F 0 "J_DC_6V_IN" H 4427 1326 50  0000 L CNN
+F 0 "J_DC_6V_IN1" H 4427 1326 50  0000 L CNN
 F 1 "Conn_01x02_Female" H 4427 1235 50  0000 L CNN
-F 2 "" H 4400 1350 50  0001 C CNN
+F 2 "Connector_PinSocket_2.54mm:PinSocket_1x02_P2.54mm_Vertical" H 4400 1350 50  0001 C CNN
 F 3 "~" H 4400 1350 50  0001 C CNN
 	1    4400 1350
@@
 	3750 1550 3750 2150
 $Comp
-L knuth:CUI_5V_SWITCHING U?
+L knuth:CUI_5V_SWITCHING U3
 U 1 1 5D1B5FD5
 P 2200 1500
-F 0 "U?" H 2031 1865 50  0000 C CNN
+F 0 "U3" H 2031 1865 50  0000 C CNN
 F 1 "CUI_5V_SWITCHING" H 2031 1774 50  0000 C CNN
-F 2 "" H 2200 1500 50  0001 C CNN
+F 2 "Connector_PinSocket_2.54mm:PinSocket_1x03_P2.54mm_Vertical" H 2200 1500 50  0001 C CNN
 F 3 "" H 2200 1500 50  0001 C CNN
 	1    2200 1500
@@
 	3950 1950 3800 1950
 $Comp
-L Connector:Conn_01x02_Female J_DC_6.5V+_IN
+L Connector:Conn_01x02_Female J_DC_6.5V+_IN1
 U 1 1 5D1BF711
 P 3150 1000
-F 0 "J_DC_6.5V+_IN" V 3090 812 50  0000 R CNN
+F 0 "J_DC_6.5V+_IN1" V 3090 812 50  0000 R CNN
 F 1 "Conn_01x02_Female" V 2999 812 50  0000 R CNN
-F 2 "" H 3150 1000 50  0001 C CNN
+F 2 "Connector_PinSocket_2.54mm:PinSocket_1x02_P2.54mm_Vertical" H 3150 1000 50  0001 C CNN
 F 3 "~" H 3150 1000 50  0001 C CNN
 	1    3150 1000
@@
 	3250 1500 3250 1200
 $Comp
-L power:GND #PWR?
+L power:GND #PWR0109
 U 1 1 5D1C288A
 P 3250 1500
-F 0 "#PWR?" H 3250 1250 50  0001 C CNN
+F 0 "#PWR0109" H 3250 1250 50  0001 C CNN
 F 1 "GND" H 3255 1327 50  0000 C CNN
 F 2 "" H 3250 1500 50  0001 C CNN
@@
 	3400 1550 3750 1550
 $Comp
-L Device:R R?
+L Device:R R2
 U 1 1 5D1CAEE6
 P 2450 1600
-F 0 "R?" V 2657 1600 50  0000 C CNN
+F 0 "R2" V 2657 1600 50  0000 C CNN
 F 1 "R" V 2566 1600 50  0000 C CNN
-F 2 "" V 2380 1600 50  0001 C CNN
+F 2 "Resistor_THT:R_Axial_DIN0204_L3.6mm_D1.6mm_P5.08mm_Horizontal" V 2380 1600 50  0001 C CNN
 F 3 "~" H 2450 1600 50  0001 C CNN
 	1    2450 1600
@@
 Wire Wire Line
 	2200 1400 3150 1400
+Wire Wire Line
+	3650 2400 3650 2950
+Wire Wire Line
+	3650 2950 4900 2950
+Connection ~ 3650 2400
+$Comp
+L Connector:Conn_01x16_Female J?
+U 1 1 5D1A8A1E
+P 1200 5400
+F 0 "J?" H 1094 4375 50  0000 C CNN
+F 1 "Conn_01x16_Female" H 1094 4466 50  0000 C CNN
+F 2 "" H 1200 5400 50  0001 C CNN
+F 3 "~" H 1200 5400 50  0001 C CNN
+	1    1200 5400
+	-1   0    0    1
+$EndComp
+Wire Wire Line
+	1850 4600 1400 4600
+Wire Wire Line
+	1400 4700 1850 4700
+Wire Wire Line
+	1850 4800 1400 4800
+Wire Wire Line
+	1400 4900 1850 4900
+Connection ~ 1850 4900
+Wire Wire Line
+	1850 5000 1400 5000
+Connection ~ 1850 5000
+Wire Wire Line
+	1400 5100 1850 5100
+Connection ~ 1850 5100
+Wire Wire Line
+	1850 5200 1400 5200
+Wire Wire Line
+	1400 5300 1850 5300
+Wire Wire Line
+	1850 5400 1400 5400
+Wire Wire Line
+	1400 5500 1850 5500
+Connection ~ 1850 5500
+Wire Wire Line
+	1850 5600 1400 5600
+Wire Wire Line
+	1400 5700 1850 5700
+Wire Wire Line
+	1850 5800 1400 5800
+Wire Wire Line
+	1400 5900 1850 5900
+Connection ~ 1850 5900
+Wire Wire Line
+	1850 6000 1400 6000
+Wire Wire Line
+	1400 6100 1850 6100
+Connection ~ 1850 6100
 $EndSCHEMATC

Commit message: update
Parts:
- J1: renamed from J?; footprint (none) -> Connector_PinSocket_2.54mm:PinSocket_1x16_P2.54mm_Vertical
- Q1: footprint (none) -> Package_TO_SOT_THT:TO-92
- Q2: footprint (none) -> Package_TO_SOT_THT:TO-220-3_Vertical
Changed lines of the file:
@@
 F 0 "Q1" H 5391 4304 50  0000 L CNN
 F 1 "Q_NPN_EBC" H 5391 4395 50  0000 L CNN
-F 2 "" H 5400 4450 50  0001 C CNN
+F 2 "Package_TO_SOT_THT:TO-92" H 5400 4450 50  0001 C CNN
 F 3 "~" H 5200 4350 50  0001 C CNN
 	1    5200 4350
@@
 F 0 "Q2" V 5628 3650 50  0000 C CNN
 F 1 "Q_NPN_BCE" V 5537 3650 50  0000 C CNN
-F 2 "" H 5500 3750 50  0001 C CNN
+F 2 "Package_TO_SOT_THT:TO-220-3_Vertical" H 5500 3750 50  0001 C CNN
 F 3 "~" H 5300 3650 50  0001 C CNN
 	1    5300 3650
@@
 Connection ~ 3650 2400
 $Comp
-L Connector:Conn_01x16_Female J?
+L Connector:Conn_01x16_Female J1
 U 1 1 5D1A8A1E
 P 1200 5400
-F 0 "J?" H 1094 4375 50  0000 C CNN
+F 0 "J1" H 1094 4375 50  0000 C CNN
 F 1 "Conn_01x16_Female" H 1094 4466 50  0000 C CNN
-F 2 "" H 1200 5400 50  0001 C CNN
+F 2 "Connector_PinSocket_2.54mm:PinSocket_1x16_P2.54mm_Vertical" H 1200 5400 50  0001 C CNN
 F 3 "~" H 1200 5400 50  0001 C CNN
 	1    1200 5400

Commit message: update
Parts:
- removed Q2: Q_NPN_BCE, Package_TO_SOT_THT:TO-220-3_Vertical, symbol Device:Q_NPN_BCE
- added Q2: Q_PNP_BCE, TO_SOT_Packages_THT:TO-220-3_Vertical, symbol device:Q_PNP_BCE
- Q1: symbol Device:Q_NPN_EBC -> knuth-gateway-rescue:Q_NPN_EBC-Device
- R1, R2, R3: symbol Device:R -> knuth-gateway-rescue:R-Device
Changed lines of the file:
@@
 $EndDescr
 $Comp
-L Device:Q_NPN_EBC Q1
+L knuth-gateway-rescue:Q_NPN_EBC-Device Q1
 U 1 1 5D1906A1
 P 5200 4350
@@
 F 3 "~" H 5200 4350 50  0001 C CNN
 	1    5200 4350
-	1    0    0    1
-$EndComp
-$Comp
-L Device:Q_NPN_BCE Q2
-U 1 1 5D1907E8
-P 5300 3650
-F 0 "Q2" V 5628 3650 50  0000 C CNN
-F 1 "Q_NPN_BCE" V 5537 3650 50  0000 C CNN
-F 2 "Package_TO_SOT_THT:TO-220-3_Vertical" H 5500 3750 50  0001 C CNN
-F 3 "~" H 5300 3650 50  0001 C CNN
-	1    5300 3650
-	0    1    -1   0
-$EndComp
-$Comp
-L Device:R R1
+	1    0    0    -1
+$EndComp
+$Comp
+L knuth-gateway-rescue:R-Device R1
 U 1 1 5D190899
 P 5300 4000
@@
 	3400 2800 4600 2800
 $Comp
-L Device:R R3
+L knuth-gateway-rescue:R-Device R3
 U 1 1 5D198BCF
 P 4050 3300
@@
 	3400 1550 3750 1550
 $Comp
-L Device:R R2
+L knuth-gateway-rescue:R-Device R2
 U 1 1 5D1CAEE6
 P 2450 1600
@@
 	1400 6100 1850 6100
 Connection ~ 1850 6100
+$Comp
+L device:Q_PNP_BCE Q2
+U 1 1 5D1BCE58
+P 5300 3650
+F 0 "Q2" V 5631 3650 50  0000 C CNN
+F 1 "Q_PNP_BCE" V 5538 3650 50  0000 C CNN
+F 2 "TO_SOT_Packages_THT:TO-220-3_Vertical" H 5500 3750 50  0001 C CNN
+F 3 "" H 5300 3650 50  0001 C CNN
+	1    5300 3650
+	0    1    -1   0
+$EndComp
 $EndSCHEMATC
