File: gateway/kg2/knuth-gateway.sch (KiCad schematic (older format))
At the start: 15 parts, among them J1 Conn_01x16_Female, Q1 Q_NPN_EBC, Q2 Q_PNP_BCE, U1 sim800, U2 Q_RHS, U3 CUI_5V_SWITCHING, U4 tpl5110, U5 adasolarlipo, U6 powerboost_1000

Commit message: update
Parts:
- R1: value R -> 500 Ohms
- R3: value R -> 1K
Changed lines of the file:
@@
 EESchema Schematic File Version 4
-EELAYER 26 0
+LIBS:knuth-gateway-cache
+EELAYER 29 0
 EELAYER END
 $Descr A4 11693 8268
@@
 P 5300 4000
 F 0 "R1" H 5370 4046 50  0000 L CNN
-F 1 "R" H 5370 3955 50  0000 L CNN
+F 1 "500 Ohms" H 5370 3955 50  0000 L CNN
 F 2 "Resistor_THT:R_Axial_DIN0204_L3.6mm_D1.6mm_P5.08mm_Horizontal" V 5230 4000 50  0001 C CNN
 F 3 "~" H 5300 4000 50  0001 C CNN
@@
 P 4050 3300
 F 0 "R3" V 3843 3300 50  0000 C CNN
-F 1 "R" V 3934 3300 50  0000 C CNN
+F 1 "1K" V 3934 3300 50  0000 C CNN
 F 2 "Resistor_THT:R_Axial_DIN0204_L3.6mm_D1.6mm_P5.08mm_Horizontal" V 3980 3300 50  0001 C CNN
 F 3 "~" H 4050 3300 50  0001 C CNN
