File: remote/kr1/_saved_knuth-gateway.sch (KiCad schematic (older format))
At the start: 9 parts, among them J1 FeatherLora1, J2 FeatherLora2, U4 tpl5110, U5 adasolarlipo

Commit message: update
Parts:
- added J?: Conn_01x02_Female, symbol Connector:Conn_01x02_Female
- R1: footprint Resistor_THT:R_Axial_DIN0309_L9.0mm_D3.2mm_P5.08mm_Vertical -> Resistor_THT:R_Axial_DIN0207_L6.3mm_D2.5mm_P5.08mm_Vertical
Changed lines of the file:
@@
 F 0 "R1" H 6380 3604 50  0000 R CNN
 F 1 "4.7K" V 6550 3750 50  0000 R CNN
-F 2 "Resistor_THT:R_Axial_DIN0309_L9.0mm_D3.2mm_P5.08mm_Vertical" V 6380 3650 50  0001 C CNN
+F 2 "Resistor_THT:R_Axial_DIN0207_L6.3mm_D2.5mm_P5.08mm_Vertical" V 6380 3650 50  0001 C CNN
 F 3 "~" H 6450 3650 50  0001 C CNN
 	1    6450 3650
@@
 Wire Wire Line
 	3550 2400 3200 2400
+$Comp
+L Connector:Conn_01x02_Female J?
+U 1 1 5D3A6032
+P 4950 2050
+F 0 "J?" H 4977 2026 50  0000 L CNN
+F 1 "Conn_01x02_Female" H 4977 1935 50  0000 L CNN
+F 2 "" H 4950 2050 50  0001 C CNN
+F 3 "~" H 4950 2050 50  0001 C CNN
+	1    4950 2050
+	1    0    0    -1
+$EndComp
 $EndSCHEMATC
