File: remote/kr1/knuth-gateway.kicad_pcb (KiCad board)
At the start: 2 copper layers, 63.5 x 64.8 mm, 15 parts, among them J1 Conn_01x16_Female, Q1 Q_NPN_EBC, Q2 Q_PNP_BCE, U1 sim800, U2 Q_RHS, U3 CUI_5V_SWITCHING, U4 tpl5110, U5 adasolarlipo, U6 powerboost_1000

Commit message: update
Parts:
- removed J_DC_6.5V+_IN1, J_DC_6V_IN1: Conn_01x02_Female, Connector_PinSocket_2.54mm:PinSocket_1x02_P2.54mm_Vertical
- removed Q1: Q_NPN_EBC, Package_TO_SOT_THT:TO-92L_Wide
- removed Q2: Q_PNP_BCE, TO_SOT_Packages_THT:TO-220-3_Vertical
- removed R2, R3: R, Resistor_THT:R_Axial_DIN0204_L3.6mm_D1.6mm_P5.08mm_Horizontal
- removed U1: sim800, Connector_PinSocket_2.54mm:PinSocket_1x12_P2.54mm_Vertical
- removed U2: Q_RHS, Connector_PinSocket_2.54mm:PinSocket_1x16_P2.54mm_Vertical
- removed U3: CUI_5V_SWITCHING, Connector_PinSocket_2.54mm:PinSocket_1x03_P2.54mm_Vertical
- removed U6: powerboost_1000, Connector_PinSocket_2.54mm:PinSocket_1x08_P2.54mm_Vertical
- added 1-Wire1: Conn_01x03_Female, Connector_PinSocket_2.54mm:PinSocket_1x03_P2.54mm_Vertical, F.Cu at (301.1, 56.4)
- added EC-5: Conn_01x03_Female, Connector_PinSocket_2.54mm:PinSocket_1x03_P2.54mm_Vertical, F.Cu at (305.7, 56.4)
- added J2: FeatherLora2, Connector_PinSocket_2.54mm:PinSocket_1x16_P2.54mm_Vertical, F.Cu at (296.5, 56.4)
- added switch1: Conn_01x03_Female, Connector_PinSocket_2.54mm:PinSocket_1x03_P2.54mm_Vertical, F.Cu at (310.3, 56.4)
- J1: value Conn_01x16_Female -> FeatherLora1; footprint Connector_PinSocket_2.54mm:PinSocket_1x16_P2.54mm_Vertical -> Connector_PinSocket_2.54mm:PinSocket_1x12_P2.54mm_Vertical
- R1: value R -> 4.7K; footprint Resistor_THT:R_Axial_DIN0204_L3.6mm_D1.6mm_P5.08mm_Horizontal -> Resistor_THT:R_Axial_DIN0309_L9.0mm_D3.2mm_P5.08mm_Vertical
Connections:
- J1 pad 1: Net-(J1-Pad1) -> VBAT
- J1 pad 10: Net-(J1-Pad10) -> D5
- J1 pad 11: Net-(J1-Pad11) -> (no net)
- J1 pad 12: Net-(J1-Pad12) -> (no net)
- J1 pad 2: Net-(J1-Pad2) -> (no net)
- J1 pad 3: Net-(J1-Pad3) -> (no net)
- J1 pad 4: Net-(J1-Pad4) -> (no net)
- J1 pad 5: Net-(J1-Pad5) -> (no net)
- J1 pad 6: Net-(J1-Pad6) -> (no net)
- J1 pad 7: GND -> D10
- J1 pad 8: Net-(J1-Pad8) -> (no net)
- J1 pad 9: Net-(J1-Pad9) -> (no net)
- R1 pad 1: Net-(Q2-Pad1) -> D5
- R1 pad 2: Net-(Q1-Pad3) -> +3V3
- U4 pad 1: +BATT -> Net-(U4-Pad1)
- U4 pad 4: Net-(R3-Pad2) -> VBAT
- U4 pad 5: Net-(J1-Pad13) -> D10
- U5 pad 1: +BATT -> Net-(U5-Pad1)
- U5 pad 3: Net-(J_DC_6V_IN1-Pad1) -> (no net)
- U5 pad 4: GND -> (no net)
Routing:
- net (no net): track 0.00 -> 132.5 mm, vias 4 -> 5
- net D10: track 0.00 -> 114.2 mm, vias 0 -> 1
- net Net-(J1-Pad13): track 106.6 -> 0.00 mm
- net Net-(J1-Pad12): track 43.1 -> 0.00 mm
- net VBAT: track 0.00 -> 33.9 mm, vias 0 -> 1
- net Net-(J1-Pad11): track 43.6 -> 18.6 mm, vias 2 -> 1
- net Net-(R3-Pad2): track 23.5 -> 0.00 mm
- net Net-(J1-Pad3): track 17.9 -> 0.00 mm
- net Net-(J_DC_6V_IN1-Pad1): track 16.1 -> 0.00 mm
- net GND: track 131.6 -> 116.8 mm, vias 6 -> 5
- net D5: track 0.00 -> 10.6 mm
- net Net-(J1-Pad1): track 110.3 -> 100.0 mm, vias 2 -> 1
- net +BATT: track 59.8 -> 53.0 mm
- net Net-(Q2-Pad1): track 5.54 -> 0.00 mm
- net Net-(J1-Pad9): track 5.08 -> 0.00 mm
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
Commit message: update
Parts:
- R1: footprint Resistor_THT:R_Axial_DIN0309_L9.0mm_D3.2mm_P5.08mm_Vertical -> Resistor_THT:R_Axial_DIN0207_L6.3mm_D2.5mm_P5.08mm_Vertical
- moved J2 80.8 mm to (238.8, 113.0), turned to 180 degrees
- moved 1-Wire1 70.6 mm to (252.7, 108.0)
- moved EC-5 66.4 mm to (252.7, 96.5)
- moved switch1 50.5 mm to (261.6, 69.8), turned to 270 degrees
- moved U5 23.0 mm to (248.9, 55.9), turned to 270 degrees
- moved R1 20.1 mm to (245.1, 108.0), turned to 270 degrees
- moved U4 10.2 mm to (252.7, 78.7)
- moved R_Delay1 9.83 mm to (246.4, 81.3)
- moved J1 5.39 mm to (218.4, 102.9)
Routing:
- net (no net): track 132.5 -> 0.00 mm, vias 5 -> 4
- net Net-(J1-Pad1): track 100.0 -> 0.00 mm, vias 1 -> 0
- net VBAT: track 33.9 -> 128.6 mm, vias 1 -> 0
- net D5: track 10.6 -> 72.1 mm, vias 0 -> 2
- net Net-(Q2-Pad2): track 57.4 -> 0.00 mm
- net +BATT: track 53.0 -> 0.00 mm
- net Net-(J_DC_6.5V+_IN1-Pad1): track 39.2 -> 0.00 mm, vias 2 -> 0
- net +3V3: track 4.37 -> 34.7 mm
- net Net-(J1-Pad11): track 18.6 -> 0.00 mm, vias 1 -> 0
- net Net-(U5-Pad1): track 0.00 -> 17.3 mm
- net A0: track 0.00 -> 16.6 mm
- net GND: track 116.8 -> 130.0 mm, vias 5 -> 0
- net Net-(U4-Pad1): track 0.00 -> 13.1 mm
- net Net-(R2-Pad1): track 9.47 -> 0.00 mm
- net D10: track 114.2 -> 121.0 mm, vias 1 -> 0
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Other:
- board size 63.5 x 64.8 mm -> 63.5 x 77.5 mm
- board text added: "Knuth Ranch: EC-5 & Temp"
- board text added: "ON/OFF"
- board text removed: "CUI"
- board text removed: "FONA 800"
- board text removed: "Knuth Ranch: Cellular Adapter"
- board text removed: "Powerboost 500"
- board text removed: "QUAHOG 0.1"

Commit message: update
Parts:
- moved 1-Wire1 3.81 mm to (252.7, 111.8)
- moved EC-5 2.54 mm to (252.7, 99.1)
Routing:
- net GND: track 130.0 -> 127.4 mm
- net +3V3: track 34.7 -> 36.9 mm
- net A0: track 16.6 -> 15.5 mm
- net D5: track 72.1 -> 71.4 mm
Other:
- board text added: "3V3"
- board text added: "A0"
- board text added: "BAT"
- board text added: "D5"
- board text added: "G"
- board text added: "[TPL5110]"
- board text added: "[feather lora]"
- board text added: "[solar lipo]"
Changed lines of the file:
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@@
   (general
     (thickness 1.6)
-    (drawings 23)
-    (tracks 77)
+    (drawings 34)
+    (tracks 73)
     (zones 0)
     (modules 9)
@@
   )
   (module Connector_PinSocket_2.54mm:PinSocket_1x03_P2.54mm_Vertical (layer F.Cu)
-    (at 252.73 107.95)
+    (at 252.73 111.76)
     (descr "Through hole straight socket strip, 1x03, 2.54mm pitch, single row (from Kicad 4.0.7), script generated")
     (tags "Through hole socket strip THT 1x03 2.54mm single row")
-    (fp_text reference 1-Wire1 (at 3.81 2.54 90) (layer F.SilkS)
+    (fp_text reference 1-Wire1 (at -3.81 2.54 90) (layer F.SilkS)
       (effects (font (size 1 1) (thickness 0.15)))
     )
@@
   )
   (module Connector_PinSocket_2.54mm:PinSocket_1x03_P2.54mm_Vertical (layer F.Cu)
-    (at 252.73 96.52)
+    (at 252.73 99.06)
     (descr "Through hole straight socket strip, 1x03, 2.54mm pitch, single row (from Kicad 4.0.7), script generated")
     (tags "Through hole socket strip THT 1x03 2.54mm single row")
-    (fp_text reference EC-5 (at 3.81 2.54 90) (layer F.SilkS)
+    (fp_text reference EC-5 (at -3.81 2.54 90) (layer F.SilkS)
       (effects (font (size 1 1) (thickness 0.15)))
     )
@@
     (descr "Resistor, Axial_DIN0207 series, Axial, Vertical, pin pitch=5.08mm, 0.25W = 1/4W, length*diameter=6.3*2.5mm^2, http://cdn-reichelt.de/documents/datenblatt/B400/1_4W%23YAG.pdf")
     (tags "Resistor Axial_DIN0207 series Axial Vertical pin pitch 5.08mm 0.25W = 1/4W length 6.3mm diameter 2.5mm")
-    (fp_text reference R1 (at 2.54 -2.37 270) (layer F.SilkS)
+    (fp_text reference R1 (at -2.54 0) (layer F.SilkS)
       (effects (font (size 1 1) (thickness 0.15)))
     )
@@
       (rotate (xyz 0 0 0))
     )
+  )
+  (gr_text [TPL5110] (at 264.414 84.2264 90) (layer F.SilkS)
+    (effects (font (size 1.5 1.5) (thickness 0.3)))
+  )
+  (gr_text "[feather lora]" (at 227.9904 84.3788 90) (layer F.SilkS)
+    (effects (font (size 1.5 1.5) (thickness 0.3)))
+  )
+  (gr_text "[solar lipo]" (at 236.1692 61.468) (layer F.SilkS)
+    (effects (font (size 1.5 1.5) (thickness 0.3)))
+  )
+  (gr_text BAT (at 249.2248 60.2996 90) (layer F.SilkS)
+    (effects (font (size 1.5 1.5) (thickness 0.3)))
+  )
+  (gr_text G (at 246.4308 59.7916 90) (layer F.SilkS)
+    (effects (font (size 1.5 1.5) (thickness 0.3)))
+  )
+  (gr_text A0 (at 256.54 99.06) (layer F.SilkS)
+    (effects (font (size 1.5 1.5) (thickness 0.3)))
+  )
+  (gr_text 3V3 (at 257.2004 101.854) (layer F.SilkS)
+    (effects (font (size 1.5 1.5) (thickness 0.3)))
+  )
+  (gr_text G (at 255.7272 104.394) (layer F.SilkS)
+    (effects (font (size 1.5 1.5) (thickness 0.3)))
+  )
+  (gr_text D5 (at 256.54 111.8108) (layer F.SilkS)
+    (effects (font (size 1.5 1.5) (thickness 0.3)))
+  )
+  (gr_text 3V3 (at 257.1496 114.5032) (layer F.SilkS)
+    (effects (font (size 1.5 1.5) (thickness 0.3)))
+  )
+  (gr_text G (at 255.9304 117.0432) (layer F.SilkS)
+    (effects (font (size 1.5 1.5) (thickness 0.3)))
   )
   (gr_text ON/OFF (at 259.08 66.548) (layer F.SilkS)
@@
   (segment (start 233.68 105.41) (end 234.95 106.68) (width 1.905) (layer B.Cu) (net 1))
   (segment (start 233.68 72.39) (end 233.68 105.41) (width 1.905) (layer B.Cu) (net 1))
-  (segment (start 247.65 101.6) (end 252.73 101.6) (width 1.905) (layer B.Cu) (net 1))
-  (segment (start 238.76 105.41) (end 243.84 105.41) (width 1.905) (layer B.Cu) (net 1))
-  (segment (start 243.84 105.41) (end 247.65 101.6) (width 1.905) (layer B.Cu) (net 1))
-  (segment (start 248.92 116.84) (end 252.73 113.03) (width 1.905) (layer B.Cu) (net 1))
   (segment (start 236.22 116.84) (end 248.92 116.84) (width 1.905) (layer B.Cu) (net 1))
   (segment (start 234.95 106.68) (end 234.95 115.57) (width 1.905) (layer B.Cu) (net 1))
   (segment (start 234.95 115.57) (end 236.22 116.84) (width 1.905) (layer B.Cu) (net 1))
   (segment (start 246.38 59.69) (end 246.38 55.88) (width 1.905) (layer B.Cu) (net 1))
+  (segment (start 248.92 116.84) (end 252.73 116.84) (width 1.905) (layer B.Cu) (net 1))
+  (segment (start 251.46 105.41) (end 238.76 105.41) (width 1.905) (layer B.Cu) (net 1))
+  (segment (start 252.73 104.14) (end 251.46 105.41) (width 1.905) (layer B.Cu) (net 1))
   (segment (start 252.73 83.82) (end 246.38 83.82) (width 1.905) (layer B.Cu) (net 2))
   (segment (start 242.57 110.49) (end 245.11 113.03) (width 1.905) (layer B.Cu) (net 3))
   (segment (start 238.76 110.49) (end 242.57 110.49) (width 1.905) (layer B.Cu) (net 3))
-  (segment (start 247.65 110.49) (end 245.11 113.03) (width 1.905) (layer B.Cu) (net 3))
-  (segment (start 252.73 110.49) (end 247.65 110.49) (width 1.905) (layer B.Cu) (net 3))
-  (segment (start 257.81 101.6) (end 255.27 99.06) (width 1.905) (layer B.Cu) (net 3))
-  (segment (start 255.27 99.06) (end 252.73 99.06) (width 1.905) (layer B.Cu) (net 3))
-  (segment (start 257.81 107.95) (end 257.81 101.6) (width 1.905) (layer B.Cu) (net 3))
-  (segment (start 252.73 110.49) (end 255.27 110.49) (width 1.905) (layer B.Cu) (net 3))
-  (segment (start 255.27 110.49) (end 257.81 107.95) (width 1.905) (layer B.Cu) (net 3))
+  (segment (start 245.11 113.03) (end 248.92 113.03) (width 1.905) (layer B.Cu) (net 3))
+  (segment (start 250.19 114.3) (end 252.73 114.3) (width 1.905) (layer B.Cu) (net 3))
+  (segment (start 248.92 113.03) (end 250.19 114.3) (width 1.905) (layer B.Cu) (net 3))
+  (segment (start 256.54 114.3) (end 252.73 114.3) (width 1.905) (layer B.Cu) (net 3))
+  (segment (start 257.81 113.03) (end 256.54 114.3) (width 1.905) (layer B.Cu) (net 3))
+  (segment (start 257.81 102.87) (end 257.81 113.03) (width 1.905) (layer B.Cu) (net 3))
+  (segment (start 252.73 101.6) (end 256.54 101.6) (width 1.905) (layer B.Cu) (net 3))
+  (segment (start 256.54 101.6) (end 257.81 102.87) (width 1.905) (layer B.Cu) (net 3))
   (segment (start 218.44 80.01) (end 219.71 80.01) (width 1.905) (layer B.Cu) (net 4))
   (segment (start 219.71 80.01) (end 229.87 90.17) (width 1.905) (layer B.Cu) (net 4))
@@
   (segment (start 229.87 115.57) (end 234.95 120.65) (width 1.905) (layer B.Cu) (net 4))
   (segment (start 234.95 120.65) (end 247.65 120.65) (width 1.905) (layer B.Cu) (net 4))
-  (segment (start 252.73 107.95) (end 251.46 106.68) (width 1.905) (layer B.Cu) (net 4))
-  (segment (start 247.65 106.68) (end 246.38 107.95) (width 1.905) (layer B.Cu) (net 4))
-  (segment (start 246.38 107.95) (end 245.11 107.95) (width 1.905) (layer B.Cu) (net 4))
-  (segment (start 248.92 106.68) (end 248.92 105.41) (width 1.905) (layer B.Cu) (net 4))
-  (segment (start 248.92 106.68) (end 247.65 106.68) (width 1.905) (layer B.Cu) (net 4))
-  (via (at 248.92 105.41) (size 1.778) (drill 0.889) (layers F.Cu B.Cu) (net 4))
-  (segment (start 251.46 106.68) (end 248.92 106.68) (width 1.905) (layer B.Cu) (net 4))
   (via (at 248.92 120.65) (size 1.778) (drill 0.889) (layers F.Cu B.Cu) (net 4))
   (segment (start 247.65 120.65) (end 248.92 120.65) (width 1.905) (layer B.Cu) (net 4))
-  (segment (start 252.73 96.52) (end 247.65 96.52) (width 1.905) (layer B.Cu) (net 5))
-  (segment (start 241.3 102.87) (end 238.76 102.87) (width 1.905) (layer B.Cu) (net 5))
-  (segment (start 247.65 96.52) (end 241.3 102.87) (width 1.905) (layer B.Cu) (net 5))
+  (via (at 248.92 107.95) (size 1.778) (drill 0.889) (layers F.Cu B.Cu) (net 4))
+  (segment (start 252.73 111.76) (end 248.92 107.95) (width 1.905) (layer B.Cu) (net 4))
+  (segment (start 248.92 107.95) (end 245.11 107.95) (width 1.905) (layer B.Cu) (net 4))
+  (segment (start 252.73 99.06) (end 246.38 99.06) (width 1.905) (layer B.Cu) (net 5))
+  (segment (start 242.57 102.87) (end 238.76 102.87) (width 1.905) (layer B.Cu) (net 5))
+  (segment (start 246.38 99.06) (end 242.57 102.87) (width 1.905) (layer B.Cu) (net 5))
   (segment (start 252.73 86.36) (end 254 86.36) (width 1.905) (layer B.Cu) (net 6))
   (segment (start 254 86.36) (end 266.7 73.66) (width 1.905) (layer B.Cu) (net 6))

Commit message: update
Parts:
- removed R1: 4.7K, Resistor_THT:R_Axial_DIN0207_L6.3mm_D2.5mm_P5.08mm_Vertical
- removed U5: adasolarlipo, Connector_PinSocket_2.54mm:PinSocket_1x04_P2.54mm_Vertical
- added RD1: R, Resistor_THT:R_Axial_DIN0207_L6.3mm_D2.5mm_P7.62mm_Horizontal, F.Cu at (250.8, 71.8)
- added RD2: R, Resistor_THT:R_Axial_DIN0207_L6.3mm_D2.5mm_P7.62mm_Horizontal, F.Cu at (245.1, 95.2)
- added RP1: 4.7K, Resistor_THT:R_Axial_DIN0207_L6.3mm_D2.5mm_P7.62mm_Horizontal, F.Cu at (245.1, 116.2)
- added solar1: Conn_01x02_Female, Connector_PinSocket_2.54mm:PinSocket_1x02_P2.54mm_Vertical, F.Cu at (249.0, 55.4)
Connections:
- J2 pad 10: (no net) -> A5
Routing:
- net A5: track 0.00 -> 28.4 mm
- net D5: track 71.4 -> 84.2 mm, vias 2 -> 0
- net D10: track 121.0 -> 113.3 mm
- net Net-(RD1-Pad1): track 17.3 -> 23.8 mm
- net GND: track 127.4 -> 133.1 mm
- net +3V3: track 36.9 -> 38.0 mm

Commit message: update
Parts:
- removed solar1: Conn_01x02_Female, Connector_PinSocket_2.54mm:PinSocket_1x02_P2.54mm_Vertical
- added J3: Conn_01x02_Female, Connector_PinSocket_2.54mm:PinSocket_1x02_P2.54mm_Vertical, F.Cu at (249.4, 65.5)
- added J4: Conn_01x02_Female, Connector_PinSocket_2.54mm:PinSocket_1x02_P2.54mm_Vertical, F.Cu at (253.5, 65.5)
- added J5: Screw_Terminal_01x03, TerminalBlock_Phoenix:TerminalBlock_Phoenix_PT-1,5-3-3.5-H_1x03_P3.50mm_Horizontal, F.Cu at (259.1, 117.9)
- added J6: Screw_Terminal_01x03, TerminalBlock_Phoenix:TerminalBlock_Phoenix_PT-1,5-3-3.5-H_1x03_P3.50mm_Horizontal, F.Cu at (259.1, 105.7)
- U4: value tpl5110 -> tpl5111
- moved RD1 6.83 mm to (244.3, 69.6), turned to 270 degrees
- moved switch1 3.87 mm to (264.5, 67.3)
Connections:
- net Net-(U4-Pad1) renamed SWITCHED_LOAD
- 1-Wire1 pad 1: D5 -> GND
- 1-Wire1 pad 3: GND -> D5
- EC-5 pad 2: +3V3 -> GND
- EC-5 pad 3: GND -> +3V3
- J1 pad 1: VBAT -> (no net)
- J1 pad 3: (no net) -> VBUS
- RD1 pad 1: Net-(RD1-Pad1) -> BATT
- U4 pad 4: VBAT -> VBUS
- switch1 pad 1: (no net) -> LOAD
- switch1 pad 3: Net-(RD1-Pad1) -> (no net)
Routing:
- net VBAT: track 128.6 -> 0.00 mm
- net VBUS: track 0.00 -> 120.9 mm
- net Net-(RD1-Pad1): track 23.8 -> 0.00 mm
- net LOAD: track 0.00 -> 14.7 mm
- net D5: track 84.2 -> 70.2 mm
- net BATT: track 0.00 -> 6.76 mm
- net A0: track 15.5 -> 22.1 mm
- net D10: track 113.3 -> 118.7 mm
- net A5: track 28.4 -> 23.4 mm
- net SWITCHED_LOAD: track 13.1 -> 16.9 mm
- net +3V3: track 38.0 -> 39.9 mm
- net GND: track 133.1 -> 131.3 mm
Other:
- board text added: "GND"
- board text added: "Knuth Ranch: REMOTE NODE + EC-5 & Temp"
- board text added: "LOAD"
- board text added: "OFF/ON"
- board text removed: "Knuth Ranch: EC-5 & Temp"
- board text removed: "ON/OFF"
