File: remote/kr1/knuth-gateway.sch (KiCad schematic (older format))
At the start: 12 parts, among them J1 Conn_01x16_Female, Q1 Q_NPN_EBC, Q2 Q_PNP_BCE, U1 sim800, U2 Q_RHS, U4 tpl5110, U5 adasolarlipo

Commit message: update
Parts:
- removed J1: Conn_01x16_Female, Connector_PinSocket_2.54mm:PinSocket_1x16_P2.54mm_Vertical, symbol knuth-gateway-rescue:Conn_01x16_Female-Connector
- removed Q1: Q_NPN_EBC, Package_TO_SOT_THT:TO-92L_Wide, symbol knuth-gateway-rescue:Q_NPN_EBC-Device
- removed Q2: Q_PNP_BCE, TO_SOT_Packages_THT:TO-220-3_Vertical, symbol knuth-gateway-rescue:Q_PNP_BCE-device
- removed R1: 500 Ohms, Resistor_THT:R_Axial_DIN0204_L3.6mm_D1.6mm_P5.08mm_Horizontal, symbol knuth-gateway-rescue:R-Device
- removed R3: 1K, Resistor_THT:R_Axial_DIN0204_L3.6mm_D1.6mm_P5.08mm_Horizontal, symbol knuth-gateway-rescue:R-Device
- removed U1: sim800, Connector_PinSocket_2.54mm:PinSocket_1x12_P2.54mm_Vertical, symbol knuth:sim800
- removed U2: Q_RHS, Connector_PinSocket_2.54mm:PinSocket_1x16_P2.54mm_Vertical, symbol knuth:Q_RHS
- added 1-Wire1, EC-5, switch1: Conn_01x03_Female, Connector_PinSocket_2.54mm:PinSocket_1x03_P2.54mm_Vertical, symbol Connector:Conn_01x03_Female
- added R1: 4.7K, Resistor_THT:R_Axial_DIN0309_L9.0mm_D3.2mm_P5.08mm_Vertical, symbol Device:R
- J1: renamed from J?; footprint (none) -> Connector_PinSocket_2.54mm:PinSocket_1x12_P2.54mm_Vertical; symbol Connector:Conn_01x12_Female -> knuth-gateway-rescue:Conn_01x12_Female-Connector
- J2: renamed from J?; footprint (none) -> Connector_PinSocket_2.54mm:PinSocket_1x16_P2.54mm_Vertical; symbol Connector:Conn_01x16_Female -> knuth-gateway-rescue:Conn_01x16_Female-Connector
Connections:
- net labels removed: +BATT
- wire segments 76 -> 31

Commit message: update
Parts:
- R1: footprint Resistor_THT:R_Axial_DIN0309_L9.0mm_D3.2mm_P5.08mm_Vertical -> Resistor_THT:R_Axial_DIN0207_L6.3mm_D2.5mm_P5.08mm_Vertical
Changed lines of the file:
@@
 EESchema Schematic File Version 4
 LIBS:knuth-gateway-cache
-EELAYER 29 0
+EELAYER 26 0
 EELAYER END
 $Descr A4 11693 8268
@@
 F 0 "R1" H 6380 3604 50  0000 R CNN
 F 1 "4.7K" V 6550 3750 50  0000 R CNN
-F 2 "Resistor_THT:R_Axial_DIN0309_L9.0mm_D3.2mm_P5.08mm_Vertical" V 6380 3650 50  0001 C CNN
+F 2 "Resistor_THT:R_Axial_DIN0207_L6.3mm_D2.5mm_P5.08mm_Vertical" V 6380 3650 50  0001 C CNN
 F 3 "~" H 6450 3650 50  0001 C CNN
 	1    6450 3650

Commit message: update
Parts:
- added J?: Conn_01x02_Female, symbol Connector:Conn_01x02_Female
Changed lines of the file:
@@
 Wire Wire Line
 	3550 2400 3200 2400
+$Comp
+L Connector:Conn_01x02_Female J?
+U 1 1 5D3A6032
+P 4950 2050
+F 0 "J?" H 4977 2026 50  0000 L CNN
+F 1 "Conn_01x02_Female" H 4977 1935 50  0000 L CNN
+F 2 "" H 4950 2050 50  0001 C CNN
+F 3 "~" H 4950 2050 50  0001 C CNN
+	1    4950 2050
+	1    0    0    -1
+$EndComp
 $EndSCHEMATC

Commit message: update
Parts:
- added RD1, RD2: R, Resistor_THT:R_Axial_DIN0207_L6.3mm_D2.5mm_P7.62mm_Horizontal, symbol Device:R
- RP1: renamed from R1; footprint Resistor_THT:R_Axial_DIN0207_L6.3mm_D2.5mm_P5.08mm_Vertical -> Resistor_THT:R_Axial_DIN0207_L6.3mm_D2.5mm_P7.62mm_Horizontal
- solar1: renamed from J?; footprint (none) -> Connector_PinSocket_2.54mm:PinSocket_1x02_P2.54mm_Vertical
Connections:
- net A5: now also RD1.2, RD2.1
- net GND: now also solar1.2 (Pin_2), RD2.2
- net at U5.1 (B+), switch1.3 (Pin_3): now also solar1.1 (Pin_1), RD1.1
Other:
- moved on the sheet: solar1
Changed lines of the file:
@@
 DI01
 Wire Wire Line
-	3800 1950 4000 1950
+	3800 1950 3950 1950
 Wire Wire Line
 	3200 2500 3750 2500
@@
 $EndComp
 $Comp
-L Device:R R1
+L Device:R RP1
 U 1 1 5D3DC753
 P 6450 3650
-F 0 "R1" H 6380 3604 50  0000 R CNN
+F 0 "RP1" H 6380 3604 50  0000 R CNN
 F 1 "4.7K" V 6550 3750 50  0000 R CNN
-F 2 "Resistor_THT:R_Axial_DIN0207_L6.3mm_D2.5mm_P5.08mm_Vertical" V 6380 3650 50  0001 C CNN
+F 2 "Resistor_THT:R_Axial_DIN0207_L6.3mm_D2.5mm_P7.62mm_Horizontal" V 6380 3650 50  0001 C CNN
 F 3 "~" H 6450 3650 50  0001 C CNN
 	1    6450 3650
@@
 U 1 1 5D40388A
 P 3550 1400
-F 0 "switch1" V 3488 1212 50  0000 R CNN
-F 1 "Conn_01x03_Female" V 3397 1212 50  0000 R CNN
+F 0 "switch1" V 3800 1600 50  0000 R CNN
+F 1 "Conn_01x03_Female" V 3650 1750 50  0000 R CNN
 F 2 "Connector_PinSocket_2.54mm:PinSocket_1x03_P2.54mm_Vertical" H 3550 1400 50  0001 C CNN
 F 3 "~" H 3550 1400 50  0001 C CNN
@@
 $EndComp
 Wire Wire Line
-	4000 1850 3650 1850
-Wire Wire Line
-	3650 1850 3650 1600
+	4000 1850 3900 1850
+Wire Wire Line
+	3650 1850 3650 1750
 Wire Wire Line
 	3550 1600 3550 2400
@@
 	3550 2400 3200 2400
 $Comp
-L Connector:Conn_01x02_Female J?
+L Connector:Conn_01x02_Female solar1
 U 1 1 5D3A6032
-P 4950 2050
-F 0 "J?" H 4977 2026 50  0000 L CNN
-F 1 "Conn_01x02_Female" H 4977 1935 50  0000 L CNN
-F 2 "" H 4950 2050 50  0001 C CNN
-F 3 "~" H 4950 2050 50  0001 C CNN
-	1    4950 2050
-	1    0    0    -1
-$EndComp
+P 4400 1450
+F 0 "solar1" H 4427 1426 50  0000 L CNN
+F 1 "Conn_01x02_Female" H 4427 1335 50  0000 L CNN
+F 2 "Connector_PinSocket_2.54mm:PinSocket_1x02_P2.54mm_Vertical" H 4400 1450 50  0001 C CNN
+F 3 "~" H 4400 1450 50  0001 C CNN
+	1    4400 1450
+	1    0    0    -1
+$EndComp
+$Comp
+L Device:R RD1
+U 1 1 5D3B9AD0
+P 2200 1900
+F 0 "RD1" H 2270 1946 50  0000 L CNN
+F 1 "R" H 2270 1855 50  0000 L CNN
+F 2 "Resistor_THT:R_Axial_DIN0207_L6.3mm_D2.5mm_P7.62mm_Horizontal" V 2130 1900 50  0001 C CNN
+F 3 "~" H 2200 1900 50  0001 C CNN
+	1    2200 1900
+	1    0    0    -1
+$EndComp
+$Comp
+L Device:R RD2
+U 1 1 5D3B9B54
+P 2200 2200
+F 0 "RD2" H 2270 2246 50  0000 L CNN
+F 1 "R" H 2270 2155 50  0000 L CNN
+F 2 "Resistor_THT:R_Axial_DIN0207_L6.3mm_D2.5mm_P7.62mm_Horizontal" V 2130 2200 50  0001 C CNN
+F 3 "~" H 2200 2200 50  0001 C CNN
+	1    2200 2200
+	1    0    0    -1
+$EndComp
+Connection ~ 3650 1750
+Wire Wire Line
+	3650 1750 3650 1600
+Wire Wire Line
+	2200 1750 3650 1750
+Wire Wire Line
+	2200 2050 2050 2050
+Connection ~ 2200 2050
+Text GLabel 2050 2050 0    50   Input ~ 0
+A5
+$Comp
+L knuth-gateway-rescue:GND-power #PWR0108
+U 1 1 5D3BB55A
+P 2200 2350
+F 0 "#PWR0108" H 2200 2100 50  0001 C CNN
+F 1 "GND" H 2205 2177 50  0000 C CNN
+F 2 "" H 2200 2350 50  0001 C CNN
+F 3 "" H 2200 2350 50  0001 C CNN
+	1    2200 2350
+	1    0    0    -1
+$EndComp
+Wire Wire Line
+	3900 1850 3900 1450
+Wire Wire Line
+	3900 1450 4200 1450
+Connection ~ 3900 1850
+Wire Wire Line
+	3900 1850 3650 1850
+Wire Wire Line
+	3950 1950 3950 1550
+Wire Wire Line
+	3950 1550 4200 1550
+Connection ~ 3950 1950
+Wire Wire Line
+	3950 1950 4000 1950
 $EndSCHEMATC

Commit message: update
Parts:
- removed U5: adasolarlipo, Connector_PinSocket_2.54mm:PinSocket_1x04_P2.54mm_Vertical, symbol knuth:adasolarlipo
- removed solar1: Conn_01x02_Female, Connector_PinSocket_2.54mm:PinSocket_1x02_P2.54mm_Vertical, symbol Connector:Conn_01x02_Female
- added J3, J4: Conn_01x02_Female, Connector_PinSocket_2.54mm:PinSocket_1x02_P2.54mm_Vertical, symbol Connector:Conn_01x02_Female
- added J5, J6: Screw_Terminal_01x03, TerminalBlock_Phoenix:TerminalBlock_Phoenix_PT-1,5-3-3.5-H_1x03_P3.50mm_Horizontal, symbol Connector:Screw_Terminal_01x03
- U4: value tpl5110 -> tpl5111
Connections:
- net +3V3: now also EC-5.3 (Pin_3), J5.2 (Pin_2), J6.1 (Pin_1); no longer EC-5.2 (Pin_2)
- net A0: now also J6.3 (Pin_3)
- net D5: now also 1-Wire1.3 (Pin_3), J5.1 (Pin_1); no longer 1-Wire1.1 (Pin_1)
- net GND: now also 1-Wire1.1 (Pin_1), EC-5.2 (Pin_2), J3.2 (Pin_2), J4.2 (Pin_2), J5.3 (Pin_3), J6.2 (Pin_2); no longer 1-Wire1.3 (Pin_3), EC-5.3 (Pin_3)
- net VBAT: no longer U4.4 (DRV)
- net VBUS: now also U4.4 (DRV)
- net SWITCHED_LOAD: now reaches U4.1 (VDD), switch1.2 (Pin_2)
- net at switch1.3 (Pin_3): no longer RD1.1
- net LOAD: now reaches switch1.1 (Pin_1)
- net LOAD: now also J4.1 (Pin_1)
- new net BATT: J3.1 (Pin_1), RD1.1
Other:
- moved on the sheet: 1-Wire1, RP1, switch1
Changed lines of the file:
@@
 P 3200 2500
 F 0 "U4" H 2956 2865 50  0000 C CNN
-F 1 "tpl5110" H 2956 2774 50  0000 C CNN
+F 1 "tpl5111" H 2956 2774 50  0000 C CNN
 F 2 "Connector_PinSocket_2.54mm:PinSocket_1x05_P2.54mm_Vertical" H 3200 2500 50  0001 C CNN
 F 3 "" H 3200 2500 50  0001 C CNN
@@
 	1    0    0    -1
 $EndComp
-$Comp
-L knuth:adasolarlipo U5
-U 1 1 5D196E31
-P 4100 1950
-F 0 "U5" H 3823 2046 50  0000 R CNN
-F 1 "adasolarlipo" H 3823 1955 50  0000 R CNN
-F 2 "Connector_PinSocket_2.54mm:PinSocket_1x04_P2.54mm_Vertical" H 4100 1950 50  0001 C CNN
-F 3 "" H 4100 1950 50  0001 C CNN
-	1    4100 1950
-	-1   0    0    -1
-$EndComp
-Wire Wire Line
-	3800 2500 3750 2500
 Connection ~ 3750 2500
 $Comp
@@
 	3300 2700 3300 3300
 Wire Wire Line
-	3800 2400 4600 2400
-Wire Wire Line
-	4600 2400 4600 2600
-Connection ~ 3800 2400
-Wire Wire Line
-	3800 2400 3800 2500
-Wire Wire Line
 	4600 2800 4600 2700
-Wire Wire Line
-	3800 1950 3800 2400
 $Comp
 L knuth-gateway-rescue:Conn_01x12_Female-Connector J1
@@
 DI01
 Wire Wire Line
-	3800 1950 3950 1950
-Wire Wire Line
 	3200 2500 3750 2500
 Wire Wire Line
@@
 P 6900 4600
 F 0 "EC-5" H 6928 4626 50  0000 L CNN
-F 1 "Conn_01x03_Female" H 6928 4535 50  0000 L CNN
+F 1 "Conn_01x03_Female" H 6600 4200 50  0000 L CNN
 F 2 "Connector_PinSocket_2.54mm:PinSocket_1x03_P2.54mm_Vertical" H 6900 4600 50  0001 C CNN
 F 3 "~" H 6900 4600 50  0001 C CNN
@@
 L Connector:Conn_01x03_Female 1-Wire1
 U 1 1 5D3CC155
-P 6900 3900
-F 0 "1-Wire1" H 6928 3926 50  0000 L CNN
-F 1 "Conn_01x03_Female" H 6928 3835 50  0000 L CNN
-F 2 "Connector_PinSocket_2.54mm:PinSocket_1x03_P2.54mm_Vertical" H 6900 3900 50  0001 C CNN
-F 3 "~" H 6900 3900 50  0001 C CNN
-	1    6900 3900
-	1    0    0    -1
-$EndComp
-Text GLabel 6650 3450 2    50   Input ~ 0
-D5
+P 6900 3800
+F 0 "1-Wire1" H 6928 3826 50  0000 L CNN
+F 1 "Conn_01x03_Female" H 6850 3450 50  0000 L CNN
+F 2 "Connector_PinSocket_2.54mm:PinSocket_1x03_P2.54mm_Vertical" H 6900 3800 50  0001 C CNN
+F 3 "~" H 6900 3800 50  0001 C CNN
+	1    6900 3800
+	1    0    0    -1
+$EndComp
 $Comp
 L knuth-gateway-rescue:GND-power #PWR0104
 U 1 1 5D3D0428
-P 6700 4000
-F 0 "#PWR0104" H 6700 3750 50  0001 C CNN
-F 1 "GND" H 6705 3827 50  0000 C CNN
-F 2 "" H 6700 4000 50  0001 C CNN
-F 3 "" H 6700 4000 50  0001 C CNN
-	1    6700 4000
-	1    0    0    -1
-$EndComp
-Text GLabel 6700 4500 0    50   Input ~ 0
+P 6400 3300
+F 0 "#PWR0104" H 6400 3050 50  0001 C CNN
+F 1 "GND" H 6405 3127 50  0000 C CNN
+F 2 "" H 6400 3300 50  0001 C CNN
+F 3 "" H 6400 3300 50  0001 C CNN
+	1    6400 3300
+	1    0    0    -1
+$EndComp
+Text GLabel 6600 4500 0    50   Input ~ 0
 A0
 $Comp
 L knuth-gateway-rescue:GND-power #PWR0105
 U 1 1 5D3D5056
-P 6700 4700
-F 0 "#PWR0105" H 6700 4450 50  0001 C CNN
-F 1 "GND" H 6705 4527 50  0000 C CNN
-F 2 "" H 6700 4700 50  0001 C CNN
-F 3 "" H 6700 4700 50  0001 C CNN
-	1    6700 4700
+P 6050 4600
+F 0 "#PWR0105" H 6050 4350 50  0001 C CNN
+F 1 "GND" H 6055 4427 50  0000 C CNN
+F 2 "" H 6050 4600 50  0001 C CNN
+F 3 "" H 6050 4600 50  0001 C CNN
+	1    6050 4600
 	1    0    0    -1
 $EndComp
@@
 L Device:R RP1
 U 1 1 5D3DC753
-P 6450 3650
-F 0 "RP1" H 6380 3604 50  0000 R CNN
-F 1 "4.7K" V 6550 3750 50  0000 R CNN
-F 2 "Resistor_THT:R_Axial_DIN0207_L6.3mm_D2.5mm_P7.62mm_Horizontal" V 6380 3650 50  0001 C CNN
-F 3 "~" H 6450 3650 50  0001 C CNN
-	1    6450 3650
+P 5900 3650
+F 0 "RP1" H 5830 3604 50  0000 R CNN
+F 1 "4.7K" V 6000 3750 50  0000 R CNN
+F 2 "Resistor_THT:R_Axial_DIN0207_L6.3mm_D2.5mm_P7.62mm_Horizontal" V 5830 3650 50  0001 C CNN
+F 3 "~" H 5900 3650 50  0001 C CNN
+	1    5900 3650
 	-1   0    0    1
 $EndComp
-Wire Wire Line
-	6700 4600 6200 4600
 $Comp
 L knuth-gateway-rescue:+3V3-power #PWR0106
@@
 	1    0    0    -1
 $EndComp
-Wire Wire Line
-	6200 3350 6200 3500
-Wire Wire Line
-	6700 3800 6650 3800
-Wire Wire Line
-	6450 3500 6200 3500
-Connection ~ 6200 3500
-Wire Wire Line
-	6200 3500 6200 3900
-Wire Wire Line
-	6650 3800 6650 3450
-Connection ~ 6650 3800
-Wire Wire Line
-	6650 3800 6450 3800
-Wire Wire Line
-	6700 3900 6200 3900
 $Comp
 L knuth-gateway-rescue:+3V3-power #PWR0107
 U 1 1 5D3F51C7
-P 6200 4600
-F 0 "#PWR0107" H 6200 4450 50  0001 C CNN
-F 1 "+3V3" H 6215 4773 50  0000 C CNN
-F 2 "" H 6200 4600 50  0001 C CNN
-F 3 "" H 6200 4600 50  0001 C CNN
-	1    6200 4600
+P 6350 4500
+F 0 "#PWR0107" H 6350 4350 50  0001 C CNN
+F 1 "+3V3" H 6365 4673 50  0000 C CNN
+F 2 "" H 6350 4500 50  0001 C CNN
+F 3 "" H 6350 4500 50  0001 C CNN
+	1    6350 4500
 	1    0    0    -1
 $EndComp
 Text GLabel 3300 3300 2    50   Input ~ 0
-VBAT
+VBUS
 Wire Wire Line
 	3200 2800 3200 3050
@@
 L Connector:Conn_01x03_Female switch1
 U 1 1 5D40388A
-P 3550 1400
-F 0 "switch1" V 3800 1600 50  0000 R CNN
-F 1 "Conn_01x03_Female" V 3650 1750 50  0000 R CNN
-F 2 "Connector_PinSocket_2.54mm:PinSocket_1x03_P2.54mm_Vertical" H 3550 1400 50  0001 C CNN
-F 3 "~" H 3550 1400 50  0001 C CNN
-	1    3550 1400
-	0    -1   -1   0
-$EndComp
-Wire Wire Line
-	4000 1850 3900 1850
-Wire Wire Line
-	3650 1850 3650 1750
-Wire Wire Line
-	3550 1600 3550 2400
-Wire Wire Line
-	3550 2400 3200 2400
-$Comp
-L Connector:Conn_01x02_Female solar1
-U 1 1 5D3A6032
-P 4400 1450
-F 0 "solar1" H 4427 1426 50  0000 L CNN
-F 1 "Conn_01x02_Female" H 4427 1335 50  0000 L CNN
-F 2 "Connector_PinSocket_2.54mm:PinSocket_1x02_P2.54mm_Vertical" H 4400 1450 50  0001 C CNN
-F 3 "~" H 4400 1450 50  0001 C CNN
-	1    4400 1450
+P 4500 1450
+F 0 "switch1" V 4750 1650 50  0000 R CNN
+F 1 "Conn_01x03_Female" V 4600 1800 50  0000 R CNN
+F 2 "Connector_PinSocket_2.54mm:PinSocket_1x03_P2.54mm_Vertical" H 4500 1450 50  0001 C CNN
+F 3 "~" H 4500 1450 50  0001 C CNN
+	1    4500 1450
 	1    0    0    -1
 $EndComp
@@
 	1    0    0    -1
 $EndComp
-Connection ~ 3650 1750
-Wire Wire Line
-	3650 1750 3650 1600
-Wire Wire Line
-	2200 1750 3650 1750
 Wire Wire Line
 	2200 2050 2050 2050
@@
 	1    0    0    -1
 $EndComp
-Wire Wire Line
-	3900 1850 3900 1450
-Wire Wire Line
-	3900 1450 4200 1450
-Connection ~ 3900 1850
-Wire Wire Line
-	3900 1850 3650 1850
-Wire Wire Line
-	3950 1950 3950 1550
-Wire Wire Line
-	3950 1550 4200 1550
-Connection ~ 3950 1950
-Wire Wire Line
-	3950 1950 4000 1950
+$Comp
+L Connector:Conn_01x02_Female J3
+U 1 1 5D3E3A64
+P 1500 850
+F 0 "J3" H 1527 826 50  0000 L CNN
+F 1 "Conn_01x02_Female" H 1527 735 50  0000 L CNN
+F 2 "Connector_PinSocket_2.54mm:PinSocket_1x02_P2.54mm_Vertical" H 1500 850 50  0001 C CNN
+F 3 "~" H 1500 850 50  0001 C CNN
+	1    1500 850
+	1    0    0    -1
+$EndComp
+$Comp
+L Connector:Conn_01x02_Female J4
+U 1 1 5D3E3B00
+P 1500 1250
+F 0 "J4" H 1527 1226 50  0000 L CNN
+F 1 "Conn_01x02_Female" H 1527 1135 50  0000 L CNN
+F 2 "Connector_PinSocket_2.54mm:PinSocket_1x02_P2.54mm_Vertical" H 1500 1250 50  0001 C CNN
+F 3 "~" H 1500 1250 50  0001 C CNN
+	1    1500 1250
+	1    0    0    -1
+$EndComp
+$Comp
+L knuth-gateway-rescue:GND-power #PWR0109
+U 1 1 5D3E3B54
+P 1300 1350
+F 0 "#PWR0109" H 1300 1100 50  0001 C CNN
+F 1 "GND" H 1305 1177 50  0000 C CNN
+F 2 "" H 1300 1350 50  0001 C CNN
+F 3 "" H 1300 1350 50  0001 C CNN
+	1    1300 1350
+	1    0    0    -1
+$EndComp
+$Comp
+L knuth-gateway-rescue:GND-power #PWR0110
+U 1 1 5D3E3BA5
+P 1300 950
+F 0 "#PWR0110" H 1300 700 50  0001 C CNN
+F 1 "GND" H 1305 777 50  0000 C CNN
+F 2 "" H 1300 950 50  0001 C CNN
+F 3 "" H 1300 950 50  0001 C CNN
+	1    1300 950
+	1    0    0    -1
+$EndComp
+Text GLabel 1300 850  0    50   Input ~ 0
+BATT
+Text GLabel 1300 1250 0    50   Input ~ 0
+LOAD
+Text GLabel 4300 1350 0    50   Input ~ 0
+LOAD
+Text GLabel 4300 1450 0    50   Input ~ 0
+SWITCHED_LOAD
+Text GLabel 3200 2400 2    50   Input ~ 0
+SWITCHED_LOAD
+Wire Wire Line
+	4600 2500 4600 2600
+Wire Wire Line
+	3750 2500 4600 2500
+Text GLabel 2200 1600 2    50   Input ~ 0
+BATT
+Wire Wire Line
+	2200 1750 2200 1600
+$Comp
+L Connector:Screw_Terminal_01x03 J5
+U 1 1 5D3E8957
+P 7450 3800
+F 0 "J5" H 7370 3475 50  0000 C CNN
+F 1 "Screw_Terminal_01x03" H 7370 3566 50  0000 C CNN
+F 2 "TerminalBlock_Phoenix:TerminalBlock_Phoenix_PT-1,5-3-3.5-H_1x03_P3.50mm_Horizontal" H 7450 3800 50  0001 C CNN
+F 3 "~" H 7450 3800 50  0001 C CNN
+	1    7450 3800
+	-1   0    0    1
+$EndComp
+$Comp
+L Connector:Screw_Terminal_01x03 J6
+U 1 1 5D3E8A32
+P 7450 4600
+F 0 "J6" H 7370 4275 50  0000 C CNN
+F 1 "Screw_Terminal_01x03" H 7370 4366 50  0000 C CNN
+F 2 "TerminalBlock_Phoenix:TerminalBlock_Phoenix_PT-1,5-3-3.5-H_1x03_P3.50mm_Horizontal" H 7450 4600 50  0001 C CNN
+F 3 "~" H 7450 4600 50  0001 C CNN
+	1    7450 4600
+	-1   0    0    1
+$EndComp
+Wire Wire Line
+	6700 3700 6550 3700
+Wire Wire Line
+	6550 3700 6550 3300
+Wire Wire Line
+	6550 3300 6400 3300
+Wire Wire Line
+	6200 3350 6200 3500
+Wire Wire Line
+	5900 3500 6200 3500
+Connection ~ 6200 3500
+Wire Wire Line
+	6200 3500 6200 3800
+Wire Wire Line
+	5900 3900 5900 3800
+Text GLabel 5800 3900 0    50   Input ~ 0
+D5
+Wire Wire Line
+	5900 3900 5800 3900
+Connection ~ 5900 3900
+Wire Wire Line
+	6200 3800 6700 3800
+Wire Wire Line
+	5900 3900 6700 3900
+Connection ~ 6700 3900
+Connection ~ 6700 3800
+Connection ~ 6700 3700
+Wire Wire Line
+	6700 4700 6350 4700
+Wire Wire Line
+	6350 4500 6350 4700
+Wire Wire Line
+	6700 4600 6050 4600
+Connection ~ 6700 4600
+Connection ~ 6700 4700
+Wire Wire Line
+	6700 4500 6600 4500
+Connection ~ 6700 4500
+Wire Wire Line
+	6700 3700 7650 3700
+Wire Wire Line
+	6700 3800 7650 3800
+Wire Wire Line
+	6700 3900 7650 3900
+Wire Wire Line
+	6700 4500 7650 4500
+Wire Wire Line
+	6700 4600 7650 4600
+Wire Wire Line
+	6700 4700 7650 4700
 $EndSCHEMATC
