File: feather_gateway/kr1/knuth-gateway.kicad_pcb (KiCad board)
At the start: 2 copper layers, 84.7 x 82.5 mm, 17 parts, among them J1 FeatherLora1, J2 FeatherLora2, J3 Conn_01x02_Female, J4 Conn_01x02_Female, J5 Conn_01x03_Female, J6 Conn_01x03_Female, J7 Conn_01x02_Female, J8 Screw_Terminal_01x03, J9 Screw_Terminal_01x03, U1 sim800, U4 tpl5111

Commit message: update
Routing:
- net GND: track 201.6 -> 199.4 mm
Other:
- board text added: "DONE"
Changed lines of the file:
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@@
   (general
     (thickness 1.6)
-    (drawings 66)
-    (tracks 230)
+    (drawings 67)
+    (tracks 229)
     (zones 0)
     (modules 17)
@@
     (descr "Resistor, Axial_DIN0207 series, Axial, Horizontal, pin pitch=10.16mm, 0.25W = 1/4W, length*diameter=6.3*2.5mm^2, http://cdn-reichelt.de/documents/datenblatt/B400/1_4W%23YAG.pdf")
     (tags "Resistor Axial_DIN0207 series Axial Horizontal pin pitch 10.16mm 0.25W = 1/4W length 6.3mm diameter 2.5mm")
-    (fp_text reference RD1 (at 5.08 -2.37 270) (layer F.SilkS)
+    (fp_text reference RD1 (at 12.7 -0.0635) (layer F.SilkS)
       (effects (font (size 1 1) (thickness 0.15)))
     )
@@
     (descr "Resistor, Axial_DIN0207 series, Axial, Horizontal, pin pitch=10.16mm, 0.25W = 1/4W, length*diameter=6.3*2.5mm^2, http://cdn-reichelt.de/documents/datenblatt/B400/1_4W%23YAG.pdf")
     (tags "Resistor Axial_DIN0207 series Axial Horizontal pin pitch 10.16mm 0.25W = 1/4W length 6.3mm diameter 2.5mm")
-    (fp_text reference RD2 (at 5.08 -2.37 90) (layer F.SilkS)
+    (fp_text reference RD2 (at -2.54 -0.0635 180) (layer F.SilkS)
       (effects (font (size 1 1) (thickness 0.15)))
     )
@@
       (rotate (xyz 0 0 0))
     )
+  )
+  (gr_text DONE (at 135.128 113.284) (layer F.SilkS)
+    (effects (font (size 1.5 1.5) (thickness 0.3)))
   )
   (gr_text 1-wire (at 143.891 138.938 90) (layer F.SilkS)
@@
   (segment (start 124.46 100.2665) (end 124.46 105.156) (width 1.905) (layer B.Cu) (net 1) (status 20))
   (segment (start 124.2695 100.076) (end 124.46 100.2665) (width 1.905) (layer B.Cu) (net 1))
-  (segment (start 124.2695 100.076) (end 122.086 100.076) (width 1.905) (layer B.Cu) (net 1))
   (segment (start 120.9675 105.156) (end 119.4435 106.68) (width 1.905) (layer B.Cu) (net 1))
   (segment (start 124.46 105.156) (end 120.9675 105.156) (width 1.905) (layer B.Cu) (net 1))

Commit message: update
Other:
- board text added: "[TPL5111]"
- board text removed: "[TPL5110]"
Changed lines of the file:
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@@
   (general
     (thickness 1.6)
-    (drawings 67)
+    (drawings 49)
     (tracks 229)
     (zones 0)
@@
     (effects (font (size 1.5 1.5) (thickness 0.3)))
   )
-  (gr_text LOAD (at 133.985 98.298) (layer F.SilkS)
-    (effects (font (size 1.5 1.5) (thickness 0.3)))
-  )
-  (gr_text BAT (at 127.635 98.298) (layer F.SilkS)
+  (gr_text LOAD (at 129.54 98.552) (layer F.SilkS)
+    (effects (font (size 1.5 1.5) (thickness 0.3)))
+  )
+  (gr_text BAT (at 122.428 98.552) (layer F.SilkS)
     (effects (font (size 1.5 1.5) (thickness 0.3)))
   )
@@
   )
   (gr_line (start 156.972 82.55) (end 74.676 82.55) (layer Edge.Cuts) (width 0.2))
-  (gr_line (start 228.1555 86.995) (end 228.092 87.0585) (layer Dwgs.User) (width 0.2))
-  (gr_line (start 228.092 90.4875) (end 228.092 87.0585) (layer Dwgs.User) (width 0.2))
-  (gr_line (start 234.1245 90.4875) (end 228.092 90.4875) (layer Dwgs.User) (width 0.2))
-  (gr_line (start 234.1245 86.995) (end 234.1245 90.4875) (layer Dwgs.User) (width 0.2))
-  (gr_line (start 228.092 86.995) (end 234.1245 86.995) (layer Dwgs.User) (width 0.2))
-  (gr_line (start 234.188 51.943) (end 228.092 51.943) (layer Dwgs.User) (width 0.2))
-  (gr_line (start 234.188 55.4355) (end 234.188 51.943) (layer Dwgs.User) (width 0.2))
-  (gr_line (start 228.092 55.4355) (end 234.188 55.4355) (layer Dwgs.User) (width 0.2))
-  (gr_line (start 228.092 51.943) (end 228.092 55.4355) (layer Dwgs.User) (width 0.2))
   (gr_text G (at 122.555 89.535) (layer F.SilkS)
     (effects (font (size 1.5 1.5) (thickness 0.3)))
-  )
-  (gr_text LOAD (at 232.41 58.801 90) (layer F.SilkS)
-    (effects (font (size 1.5 1.5) (thickness 0.3)))
-  )
-  (dimension 7.493 (width 0.3) (layer Dwgs.User)
-    (gr_text "7.493 mm" (at 236.2835 37.27) (layer Dwgs.User)
-      (effects (font (size 1.5 1.5) (thickness 0.3)))
-    )
-    (feature1 (pts (xy 232.537 61.595) (xy 232.537 38.783579)))
-    (feature2 (pts (xy 240.03 61.595) (xy 240.03 38.783579)))
-    (crossbar (pts (xy 240.03 39.37) (xy 232.537 39.37)))
-    (arrow1a (pts (xy 232.537 39.37) (xy 233.663504 38.783579)))
-    (arrow1b (pts (xy 232.537 39.37) (xy 233.663504 39.956421)))
-    (arrow2a (pts (xy 240.03 39.37) (xy 238.903496 38.783579)))
-    (arrow2b (pts (xy 240.03 39.37) (xy 238.903496 39.956421)))
   )
   (dimension 20.32 (width 0.3) (layer Dwgs.User)
@@
     (arrow2b (pts (xy 82.539285 139.114109) (xy 83.665789 138.527688)))
   )
-  (gr_text [TPL5110] (at 141.859 108.3564 90) (layer F.SilkS)
+  (gr_text [TPL5111] (at 141.859 108.3564 90) (layer F.SilkS)
     (effects (font (size 1.5 1.5) (thickness 0.3)))
   )
@@
     (effects (font (size 1.5 1.5) (thickness 0.3)))
   )
-  (gr_text BAT (at 232.791 84.455 90) (layer F.SilkS)
-    (effects (font (size 1.5 1.5) (thickness 0.3)))
-  )
-  (gr_text G (at 229.362 85.471 90) (layer F.SilkS)
-    (effects (font (size 1.5 1.5) (thickness 0.3)))
-  )
   (gr_text A0 (at 130.81 123.317) (layer F.SilkS)
     (effects (font (size 1.5 1.5) (thickness 0.3)))
@@
     (effects (font (size 1.5 1.5) (thickness 0.3)))
   )
-  (dimension 40.64 (width 0.3) (layer Dwgs.User)
-    (gr_text "1.6000 in" (at 219.71 46.16) (layer Dwgs.User)
-      (effects (font (size 1.5 1.5) (thickness 0.3)))
-    )
-    (feature1 (pts (xy 240.03 50.8) (xy 240.03 47.673579)))
-    (feature2 (pts (xy 199.39 50.8) (xy 199.39 47.673579)))
-    (crossbar (pts (xy 199.39 48.26) (xy 240.03 48.26)))
-    (arrow1a (pts (xy 240.03 48.26) (xy 238.903496 48.846421)))
-    (arrow1b (pts (xy 240.03 48.26) (xy 238.903496 47.673579)))
-    (arrow2a (pts (xy 199.39 48.26) (xy 200.516504 48.846421)))
-    (arrow2b (pts (xy 199.39 48.26) (xy 200.516504 47.673579)))
-  )
-  (gr_line (start 240.03 91.44) (end 240.03 50.8) (layer Dwgs.User) (width 0.2))
-  (gr_line (start 199.39 91.44) (end 240.03 91.44) (layer Dwgs.User) (width 0.2))
-  (gr_line (start 199.39 50.8) (end 199.39 91.44) (layer Dwgs.User) (width 0.2))
-  (gr_line (start 240.03 50.8) (end 199.39 50.8) (layer Dwgs.User) (width 0.2))
   (gr_text pvos.org/knuth (at 295.91 106.68 90) (layer F.SilkS)
     (effects (font (size 1.5 1.5) (thickness 0.3)))
