File: remote/kr2/knuth-gateway.kicad_pcb (KiCad board)
At the start: 2 copper layers, 69.1 x 80.6 mm, 21 parts, among them J1 FeatherLora1, J10 Screw_Terminal_01x02, J11 Screw_Terminal_01x02, J2 FeatherLora2, J3 Conn_01x02_Female, J4 Conn_01x02_Female, J5 Screw_Terminal_01x03, J6 Screw_Terminal_01x03, J7 Conn_01x03_Female, J8 Conn_01x02_Female, J9 Conn_01x02_Female, U4 tpl5111

Commit message: update
Routing:
- net GND: track 254.9 -> 257.2 mm
- net EXT_BAT: track 60.8 -> 60.1 mm
Changed lines of the file:
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@@
     (thickness 1.6)
     (drawings 31)
-    (tracks 176)
+    (tracks 179)
     (zones 0)
     (modules 21)
@@
   (segment (start 245.11 105.41) (end 245.11 102.87) (width 1.905) (layer B.Cu) (net 1) (status 20))
   (segment (start 245.11 105.41) (end 238.76 105.41) (width 1.905) (layer B.Cu) (net 1) (status 20))
-  (segment (start 246.38 101.6) (end 245.11 102.87) (width 1.905) (layer B.Cu) (net 1) (status 20))
-  (segment (start 252.73 101.6) (end 246.38 101.6) (width 1.905) (layer B.Cu) (net 1) (status 10))
   (segment (start 253.634 110.856) (end 252.73 111.76) (width 1.905) (layer B.Cu) (net 1) (status 20))
   (segment (start 259.08 110.856) (end 253.634 110.856) (width 1.905) (layer B.Cu) (net 1) (status 10))
@@
   (segment (start 247.396 79.248) (end 247.396 76.2) (width 1.905) (layer B.Cu) (net 1))
   (segment (start 234.95 105.41) (end 238.76 105.41) (width 1.905) (layer B.Cu) (net 1))
-  (segment (start 253.912001 50.902501) (end 242.149999 50.902501) (width 1.905) (layer B.Cu) (net 1))
   (segment (start 254.762 51.7525) (end 253.912001 50.902501) (width 1.905) (layer B.Cu) (net 1))
-  (segment (start 241.808 51.2445) (end 241.808 54.4195) (width 1.905) (layer B.Cu) (net 1))
-  (segment (start 242.149999 50.902501) (end 241.808 51.2445) (width 1.905) (layer B.Cu) (net 1))
-  (segment (start 241.808 54.4195) (end 241.808 53.217419) (width 1.905) (layer B.Cu) (net 1))
   (segment (start 263.525 52.5145) (end 263.525 50.7365) (width 1.905) (layer B.Cu) (net 1))
   (segment (start 263.525 50.7365) (end 261.62 48.8315) (width 1.905) (layer B.Cu) (net 1))
@@
   (segment (start 225.806 49.3395) (end 228.346 51.8795) (width 1.905) (layer B.Cu) (net 1))
   (segment (start 219.964 49.3395) (end 225.806 49.3395) (width 1.905) (layer B.Cu) (net 1))
-  (segment (start 241.173 51.8795) (end 242.149999 50.902501) (width 1.905) (layer B.Cu) (net 1))
-  (segment (start 228.346 51.8795) (end 241.173 51.8795) (width 1.905) (layer B.Cu) (net 1))
   (segment (start 245.745 73.025) (end 249.428 69.342) (width 1.905) (layer B.Cu) (net 1))
   (segment (start 245.745 74.549) (end 245.745 73.025) (width 1.905) (layer B.Cu) (net 1))
@@
   (segment (start 265.3665 56.0705) (end 271.78 62.484) (width 1.905) (layer B.Cu) (net 1))
   (segment (start 263.976 56.0705) (end 265.3665 56.0705) (width 1.905) (layer B.Cu) (net 1))
+  (segment (start 251.527919 101.6) (end 250.257919 102.87) (width 1.905) (layer B.Cu) (net 1))
+  (segment (start 252.73 101.6) (end 251.527919 101.6) (width 1.905) (layer B.Cu) (net 1))
+  (segment (start 250.257919 102.87) (end 245.11 102.87) (width 1.905) (layer B.Cu) (net 1))
+  (segment (start 229.195999 51.029501) (end 229.195999 50.966001) (width 1.905) (layer B.Cu) (net 1))
+  (segment (start 228.346 51.8795) (end 229.195999 51.029501) (width 1.905) (layer B.Cu) (net 1))
+  (segment (start 229.195999 50.966001) (end 230.505 49.657) (width 1.905) (layer B.Cu) (net 1))
+  (segment (start 252.6665 49.657) (end 254.762 51.7525) (width 1.905) (layer B.Cu) (net 1))
+  (segment (start 241.681 53.090419) (end 241.681 49.657) (width 1.905) (layer B.Cu) (net 1))
+  (segment (start 230.505 49.657) (end 241.681 49.657) (width 1.905) (layer B.Cu) (net 1))
+  (segment (start 241.808 53.217419) (end 241.681 53.090419) (width 1.905) (layer B.Cu) (net 1))
+  (segment (start 241.808 54.4195) (end 241.808 53.217419) (width 1.905) (layer B.Cu) (net 1))
+  (segment (start 241.681 49.657) (end 252.6665 49.657) (width 1.905) (layer B.Cu) (net 1))
   (segment (start 252.73 83.82) (end 246.38 83.82) (width 1.905) (layer B.Cu) (net 2) (status 30))
   (segment (start 243.205 110.49) (end 245.11 108.585) (width 1.905) (layer B.Cu) (net 3) (status 20))
@@
   (segment (start 254.762 54.2925) (end 258.247 54.2925) (width 1.905) (layer B.Cu) (net 13))
   (segment (start 216.789 59.182) (end 211.709 64.262) (width 1.905) (layer B.Cu) (net 13))
-  (segment (start 242.404 60.198) (end 229.87 60.198) (width 1.905) (layer B.Cu) (net 13))
   (segment (start 211.709 64.262) (end 211.709 68.834) (width 1.905) (layer B.Cu) (net 13))
-  (segment (start 229.87 60.198) (end 228.854 59.182) (width 1.905) (layer B.Cu) (net 13))
   (segment (start 228.854 59.182) (end 216.789 59.182) (width 1.905) (layer B.Cu) (net 13))
-  (segment (start 242.404 60.198) (end 242.404 59.6655) (width 1.905) (layer B.Cu) (net 13))
   (segment (start 244.348 57.7215) (end 244.348 54.4195) (width 1.905) (layer B.Cu) (net 13))
   (segment (start 242.404 59.6655) (end 244.348 57.7215) (width 1.905) (layer B.Cu) (net 13))
+  (segment (start 229.3375 59.6655) (end 228.854 59.182) (width 1.905) (layer B.Cu) (net 13))
+  (segment (start 242.404 59.6655) (end 229.3375 59.6655) (width 1.905) (layer B.Cu) (net 13))
   (segment (start 223.393 54.4195) (end 228.346 54.4195) (width 1.905) (layer B.Cu) (net 14))
   (segment (start 221.869 52.8955) (end 223.393 54.4195) (width 1.905) (layer B.Cu) (net 14))

Commit message: update
Parts:
- moved switch1 1.85 mm to (266.4, 67.4)
- moved J4 1.18 mm to (255.4, 66.8)
Routing:
- net GND: track 257.2 -> 263.9 mm
- net VBUS: track 127.9 -> 131.7 mm
- net LOAD: track 14.4 -> 16.9 mm
- net SWITCHED_LOAD: track 16.9 -> 17.7 mm
Other:
- board size 69.1 x 80.6 mm -> 72.8 x 83.6 mm
- board text added: "5VOUT"
- board text added: "DELAY"
- board text added: "DONE"
- board text added: "DRV"
- board text added: "VDD"
- board text added: "VEXT"
- board text removed: "[solar lipo]"
