File: feather_gateway/kr2/knuth-gateway.sch (KiCad schematic (older format))
At the start: 24 parts, among them J1 FeatherLora1, J11 Conn_01x02_Female, J12 Conn_01x02_Female, J2 FeatherLora2, J3 Conn_01x02_Female, J4 Conn_01x02_Female, J5 Conn_01x03_Female, J6 Conn_01x03_Female, J7 Conn_01x02_Female, J8 Screw_Terminal_01x03, J9 Screw_Terminal_01x03, U1 sim800, U4 tpl5111

Commit message: update
Changed lines of the file:
@@
 Text GLabel 3150 1500 0    50   Input ~ 0
 EXT_BAT
-Text GLabel 3150 1600 0    50   Input ~ 0
-GND
 Text GLabel 3150 1700 0    50   Input ~ 0
 5V_OUT
@@
 	3500 1700 3150 1700
 Connection ~ 3350 1600
-Wire Wire Line
-	3350 1600 3150 1600
 Wire Wire Line
 	3350 2100 4250 2100
@@
 Wire Wire Line
 	6650 850  6650 700
+Wire Wire Line
+	2650 1600 2650 1650
+Wire Wire Line
+	2650 1600 3350 1600
+$Comp
+L power:GND #PWR?
+U 1 1 5D40C0D2
+P 2650 1650
+F 0 "#PWR?" H 2650 1400 50  0001 C CNN
+F 1 "GND" H 2655 1477 50  0000 C CNN
+F 2 "" H 2650 1650 50  0001 C CNN
+F 3 "" H 2650 1650 50  0001 C CNN
+	1    2650 1650
+	1    0    0    -1
+$EndComp
 $EndSCHEMATC
